File: PCBs/haptic display/haptic display 8x8/haptic display 8x8 driver/haptic display 8x8 driver.kicad_pcb (KiCad board)
At the start: 2 copper layers, 145 x 145 mm, 20 parts, among them IC1 DRV8912QPWPRQ1, IC2 DRV8912QPWPRQ1, IC3 DRV8912QPWPRQ1, J1 UJC-HP-3-SMT-TR, J2 Conn_01x08_Female, J3 Conn_01x08_Female, J4 Conn_01x08_Female, J5 Conn_01x08_Female, U1 WeMos_D1_mini

Commit message: cleanup
Connections:
- U1 pad 10: Net-(U1-Pad10) -> GND
Routing:
- net GND: track 0.00 -> 29.1 mm
- net /c8_f: track 100.7 -> 102.8 mm
- net /r6_b: track 85.1 -> 87.2 mm
- net /r5_b: track 91.0 -> 92.8 mm
- net /r1_b: track 98.3 -> 99.8 mm
- net /r2_b: track 79.3 -> 80.3 mm
Other:
- board text added: "haptic display 8x8 driver v2"
- board text removed: "haptic display 8x8 driver v1"
