File: PCBs/haptic display/haptic display 8x8/haptic display 8x8 driver/haptic display 8x8 driver.sch (KiCad schematic (older format))
At the start: 20 parts, among them IC1 DRV8912QPWPRQ1, IC2 DRV8912QPWPRQ1, IC3 DRV8912QPWPRQ1, J1 UJC-HP-3-SMT-TR, J2 Conn_01x08_Female, J3 Conn_01x08_Female, J4 Conn_01x08_Female, J5 Conn_01x08_Female, U1 WeMos_D1_mini

Commit message: cleanup
Connections:
- net GND: now also U1.10 (GND)
Changed lines of the file:
@@
 	1    0    0    -1
 $EndComp
+$Comp
+L power:GND #PWR?
+U 1 1 60289CCF
+P 1850 5200
+F 0 "#PWR?" H 1850 4950 50  0001 C CNN
+F 1 "GND" H 1855 5027 50  0000 C CNN
+F 2 "" H 1850 5200 50  0001 C CNN
+F 3 "" H 1850 5200 50  0001 C CNN
+	1    1850 5200
+	1    0    0    -1
+$EndComp
+Wire Wire Line
+	1850 4950 1850 5200
 $EndSCHEMATC
